Commit message: reduce torque limits

File: src/sew_agv_description/urdf/sew_agv_gazebo_macro.urdf.xacro (robot description, xacro)
@@ -14,6 +14,6 @@
                 <wheel_diameter>0.2</wheel_diameter>
                 <!-- joint limits/ overrides urdf definitions ! -->
-                <max_wheel_torque>200</max_wheel_torque>
-                <max_wheel_acceleration>10.0</max_wheel_acceleration>
+                <max_wheel_torque>20</max_wheel_torque>
+                <max_wheel_acceleration>1.0</max_wheel_acceleration>
                 <!-- Output messages of the plugin gazebo -> ros2-->
                 <odometry_frame>odom</odometry_frame>

File: src/sew_agv_description/urdf/sew_agv_macro.urdf.xacro (robot description, xacro)
@@ -81,5 +81,5 @@
         <origin rpy="1.57079 0 0" xyz="0.290 0 -0.56"/>
         <axis xyz="0 0 1"/>
-        <limit effort="1000.0" velocity="3.5"/>    <!--effort in Nm, velocity in m/s-->
+        <limit effort="10.0" velocity="3.5"/>    <!--effort in Nm, velocity in m/s-->
         <parent link="base_link"/>
         <child link="caster_wheel_link"/>
@@ -108,5 +108,5 @@
     <joint name="wheel_right_joint" type="continuous">
         <origin rpy="0 0 -1.57079" xyz="-0.225 -0.2625 -0.48"/>
-        <limit effort="1000.0" velocity="3.5"/>
+        <limit effort="10.0" velocity="3.5"/>
         <axis xyz="-1 0 0"/>
         <parent link="base_link"/>
@@ -137,5 +137,5 @@
     <joint name="wheel_left_joint" type="continuous">
         <origin rpy="0 0 1.57079" xyz="-0.225 0.2625 -0.48"/>
-        <limit effort="1000.0" velocity="3.5"/>
+        <limit effort="10.0" velocity="3.5"/>
         <axis xyz="1 0 0"/>
         <parent link="base_link"/>

Commit message: add lidar plugin and relocate scanner joint

File: src/sew_agv_description/urdf/sew_agv_gazebo_macro.urdf.xacro (robot description, xacro)
@@ -51,4 +51,34 @@
             <mu2 value="0.001"/>
         </gazebo>
+    <!--#######################################################################################################################################-->
+    <!--include lidar sensor simulation on lidar link -->
+    <!--#######################################################################################################################################-->
+        <gazebo reference="lidar_link">
+            <sensor type="ray" name="lidar_1">
+                <pose> 0 0 0 0 0 0 </pose>      <!--define offset to lidar_link frame-->
+                <visualize>true</visualize>
+                <update_rate>10</update_rate>
+                <ray>                               <!--define field of view-->
+                    <scan>
+                        <horizontal>
+                            <samples>720</samples>
+                            <min_angle>-2</min_angle>
+                            <max_angle>2</max_angle>
+                        </horizontal>
+                    </scan>
+                    <range>
+                        <min>0.3</min>
+                        <max>5</max>
+                    </range>
+                </ray>
+                <plugin name="laser_controller" filename="libgazebo_ros_ray_sensor.so">     <!--call gazebo plugin for lidar-->
+                    <ros>
+                        <argument>~/out:=scan</argument>        <!--define output topic-->
+                    </ros>
+                    <output_type>sensor_msgs/LaserScan</output_type>
+                    <frame_name>lidar_link</frame_name>
+                </plugin>
+            </sensor>
+        </gazebo>
     </xacro:macro>
 </robot>

File: src/sew_agv_description/urdf/sew_agv_macro.urdf.xacro (robot description, xacro)
@@ -165,5 +165,5 @@
     <joint name="lidar_joint" type="fixed">
         <axis xyz="0 0 0"/>
-        <origin rpy="0 0 0 " xyz="0.355 0 -0.465"/>
+        <origin rpy="0 0 0 " xyz="0.355 0 -0.445"/>
         <parent link="base_link"/>
         <child link="lidar_link"/>

Commit message: add tf prefix as parameter

File: src/sew_agv_description/urdf/sew_agv_gazebo_macro.urdf.xacro (robot description, xacro)
@@ -1,5 +1,5 @@
 <?xml version="1.0"?>
 <robot xmlns:xacro="http://www.ros.org/wiki/xacro">
-    <xacro:macro name="sew_agv_gazebo">
+    <xacro:macro name="sew_agv_gazebo" params="tf_prefix">
     <!--#######################################################################################################################################-->
     <!--set up the diff_drive plugin controller from gazebo, NOT ros2_control -> maybe change when ros2_control available -->
@@ -30,17 +30,17 @@
     <!--define gazebo tags for materials, because urdf materialc can not be used in gazebo -->
     <!--#######################################################################################################################################-->
-        <gazebo reference="sew_caster_wheel_link">
+        <gazebo reference="${tf_prefix}caster_wheel_link">
             <material> Gazebo/Black</material>
         </gazebo>
-        <gazebo reference="sew_right_wheel_link">
+        <gazebo reference="${tf_prefix}right_wheel_link">
             <material> Gazebo/Black</material>
         </gazebo>
-        <gazebo reference="sew_left_wheel_link">
+        <gazebo reference="${tf_prefix}left_wheel_link">
             <material> Gazebo/Black</material>
         </gazebo>
-        <gazebo reference="sew_body_link">
+        <gazebo reference="${tf_prefix}body_link">
             <material> Gazebo/Grey</material>
         </gazebo>
-        <gazebo reference="sew_lidar_link">
+        <gazebo reference="${tf_prefix}lidar_link">
             <material> Gazebo/Yellow</material>
         </gazebo>
@@ -48,5 +48,5 @@
     <!--set friction of the caster wheel to nearly 0 (for simplicity reasons) -->
     <!--#######################################################################################################################################-->
-        <gazebo reference="sew_caster_wheel_link">
+        <gazebo reference="${tf_prefix}caster_wheel_link">
             <mu1 value="0.001"/>
             <mu2 value="0.001"/>
@@ -55,5 +55,5 @@
     <!--include lidar sensor simulation on lidar link -->
     <!--#######################################################################################################################################-->
-        <gazebo reference="sew_lidar_link">
+        <gazebo reference="${tf_prefix}lidar_link">
             <sensor type="ray" name="lidar_1">
                 <pose> 0 0 0 0 0 0 </pose>      <!--define offset to lidar_link frame-->

File: src/sew_agv_description/urdf/sew_agv_macro.urdf.xacro (robot description, xacro)
@@ -35,5 +35,5 @@
     <xacro:if value="${standalone_gazebo}">
         <xacro:include filename="$(find sew_agv_description)/urdf/sew_agv_gazebo_macro.urdf.xacro" />
-        <xacro:sew_agv_gazebo/>
+        <xacro:sew_agv_gazebo tf_prefix="${tf_prefix}"/>
     </xacro:if>
 <!--#######################################################################################################################################-->
@@ -42,5 +42,5 @@
     <xacro:if value="${ros2_control_with_gazebo}">
         <xacro:include filename="$(find sew_agv_description)/urdf/sew_agv_ros2_control_gazebo_macro.urdf.xacro" />
-        <xacro:sew_ros2_control_gazebo/>
+        <xacro:sew_ros2_control_gazebo tf_prefix="${tf_prefix}"/>
     </xacro:if>
 <!--#######################################################################################################################################-->

File: src/sew_agv_description/urdf/sew_agv_ros2_control_gazebo_macro.urdf.xacro (robot description, xacro)
@@ -1,5 +1,5 @@
 <?xml version="1.0"?>
 <robot xmlns:xacro="http://www.ros.org/wiki/xacro">
-    <xacro:macro name="sew_ros2_control_gazebo">
+    <xacro:macro name="sew_ros2_control_gazebo" params="tf_prefix">
     <!--#######################################################################################################################################-->
     <!--set up the ros2 control plugin for the sew diff drive controller-->
@@ -14,7 +14,32 @@
     </gazebo>
     <!--#######################################################################################################################################-->
+    <!--define gazebo tags for materials, because urdf materialc can not be used in gazebo -->
+    <!--#######################################################################################################################################-->
+        <gazebo reference="${tf_prefix}caster_wheel_link">
+            <material> Gazebo/Black</material>
+        </gazebo>
+        <gazebo reference="${tf_prefix}right_wheel_link">
+            <material> Gazebo/Black</material>
+        </gazebo>
+        <gazebo reference="${tf_prefix}left_wheel_link">
+            <material> Gazebo/Black</material>
+        </gazebo>
+        <gazebo reference="${tf_prefix}body_link">
+            <material> Gazebo/Grey</material>
+        </gazebo>
+        <gazebo reference="${tf_prefix}lidar_link">
+            <material> Gazebo/Yellow</material>
+        </gazebo>
+    <!--#######################################################################################################################################-->
+    <!--set friction of the caster wheel to nearly 0 (for simplicity reasons) -->
+    <!--#######################################################################################################################################-->
+        <gazebo reference="${tf_prefix}caster_wheel_link">
+            <mu1 value="0.001"/>
+            <mu2 value="0.001"/>
+        </gazebo>
+    <!--#######################################################################################################################################-->
     <!--include lidar sensor simulation on lidar link -->
     <!--#######################################################################################################################################-->
-        <gazebo reference="sew_lidar_link">
+        <gazebo reference="${tf_prefix}lidar_link">
             <sensor type="ray" name="lidar_1">
                 <pose> 0 0 0 0 0 0 </pose>      <!--define offset to lidar_link frame-->
