Commit message: redo paths to absolute paths --> gazebo works, but rviz not

File: src/sew_agv_description/urdf/sew_agv_macro.urdf.xacro (robot description, xacro)
@@ -65,5 +65,5 @@
             <origin rpy="0 0 0" xyz="0 0 0"/>
             <geometry>
-                <mesh filename="package://sew_agv_description/meshes/visual/sew_maxo_mts_body.stl" scale="0.001 0.001 0.001"/>
+                <mesh filename="/home/logilab/ros2_ws/src/sew_agv_description/meshes/visual/sew_maxo_mts_body.stl" scale="0.001 0.001 0.001"/>
             </geometry>
             <material name="${tf_prefix}grey"/>
@@ -72,5 +72,5 @@
             <origin rpy=" 0 0 0" xyz="0 0 0"/>
             <geometry>
-                <mesh filename="package://sew_agv_description/meshes/collision/sew_maxo_mts_body.stl" scale="0.001 0.001 0.001"/>
+                <mesh filename="/home/logilab/ros2_ws/src/sew_agv_description/meshes/collision/sew_maxo_mts_body.stl" scale="0.001 0.001 0.001"/>
             </geometry>
             <material name="${tf_prefix}red"/>
@@ -93,5 +93,5 @@
             <origin rpy="0 0 0" xyz="0 0 0"/>
             <geometry>
-                <mesh filename="package://sew_agv_description/meshes/visual/sew_maxo_mts_front_wheel.stl" scale="0.001 0.001 0.001"/>
+                <mesh filename="/home/logilab/ros2_ws/src/sew_agv_description/meshes/visual/sew_maxo_mts_front_wheel.stl" scale="0.001 0.001 0.001"/>
             </geometry>
             <material name="${tf_prefix}black"/>
@@ -100,5 +100,5 @@
             <origin rpy="0 0 0" xyz="0 0 0"/>
             <geometry>
-                <mesh filename="package://sew_agv_description/meshes/visual/sew_maxo_mts_front_wheel.stl" scale="0.001 0.001 0.001"/>
+                <mesh filename="/home/logilab/ros2_ws/src/sew_agv_description/meshes/visual/sew_maxo_mts_front_wheel.stl" scale="0.001 0.001 0.001"/>
             </geometry>
             <material name="${tf_prefix}red"/>
@@ -122,5 +122,5 @@
             <origin rpy="0 0 0" xyz="0 0 0"/>
             <geometry>
-                <mesh filename="package://sew_agv_description/meshes/visual/sew_maxo_mts_wheel.stl" scale="0.001 0.001 0.001"/>
+                <mesh filename="/home/logilab/ros2_ws/src/sew_agv_description/meshes/visual/sew_maxo_mts_wheel.stl" scale="0.001 0.001 0.001"/>
             </geometry>
             <material name="${tf_prefix}black"/>
@@ -129,5 +129,5 @@
             <origin rpy="0 0 0" xyz="0 0 0"/>
             <geometry>
-                <mesh filename="package://sew_agv_description/meshes/visual/sew_maxo_mts_wheel.stl" scale="0.001 0.001 0.001"/>
+                <mesh filename="/home/logilab/ros2_ws/src/sew_agv_description/meshes/visual/sew_maxo_mts_wheel.stl" scale="0.001 0.001 0.001"/>
             </geometry>
             <material name="${tf_prefix}red"/>
@@ -151,5 +151,5 @@
             <origin rpy="0 0 0" xyz="0 0 0"/>
             <geometry>
-                <mesh filename="package://sew_agv_description/meshes/visual/sew_maxo_mts_wheel.stl" scale="0.001 0.001 0.001"/>
+                <mesh filename="/home/logilab/ros2_ws/src/sew_agv_description/meshes/visual/sew_maxo_mts_wheel.stl" scale="0.001 0.001 0.001"/>
             </geometry>
             <material name="${tf_prefix}black"/>
@@ -158,5 +158,5 @@
             <origin rpy="0 0 0" xyz="0 0 0"/>
             <geometry>
-                <mesh filename="package://sew_agv_description/meshes/visual/sew_maxo_mts_wheel.stl" scale="0.001 0.001 0.001"/>
+                <mesh filename="/home/logilab/ros2_ws/src/sew_agv_description/meshes/visual/sew_maxo_mts_wheel.stl" scale="0.001 0.001 0.001"/>
             </geometry>
             <material name="${tf_prefix}red"/>
@@ -179,5 +179,5 @@
             <origin rpy="0 0 0" xyz="0 0 0"/>
             <geometry>
-                <mesh filename="package://sew_agv_description/meshes/visual/sew_maxo_mts_lidar.stl" scale="0.001 0.001 0.001"/>
+                <mesh filename="/home/logilab/ros2_ws/src/sew_agv_description/meshes/visual/sew_maxo_mts_lidar.stl" scale="0.001 0.001 0.001"/>
             </geometry>
             <material name="${tf_prefix}yellow"/>
@@ -186,5 +186,5 @@
             <origin rpy="0 0 0" xyz="0 0 0"/>
             <geometry>
-                <mesh filename="package://sew_agv_description/meshes/visual/sew_maxo_mts_lidar.stl" scale="0.001 0.001 0.001"/>
+                <mesh filename="/home/logilab/ros2_ws/src/sew_agv_description/meshes/visual/sew_maxo_mts_lidar.stl" scale="0.001 0.001 0.001"/>
             </geometry>
         </collision>

Commit message: change axis in urdf

File: src/sew_agv_description/urdf/sew_agv_macro.urdf.xacro (robot description, xacro)
@@ -52,5 +52,5 @@
     <joint name="base_footprint_joint" type="fixed">
         <origin rpy="0 0 0" xyz="0 0 0.58"/>
-        <axis xyz="0 0 1"/>
+        <axis xyz="0 0 0"/>
         <parent link="base_footprint"/>
         <child link="base_link"/>
@@ -80,6 +80,5 @@
     <joint name="caster_wheel_joint" type="fixed">
         <origin rpy="1.57079 0 0" xyz="0.290 0 -0.56"/>
-        <axis xyz="0 0 1"/>
-        <limit effort="10.0" velocity="3.5"/>    <!--effort in Nm, velocity in m/s-->
+        <axis xyz="0 0 0"/>
         <parent link="base_link"/>
         <child link="caster_wheel_link"/>
@@ -108,5 +107,5 @@
     <joint name="wheel_right_joint" type="continuous">
         <origin rpy="0 0 -1.57079" xyz="-0.225 -0.2625 -0.48"/>
-        <limit effort="10.0" velocity="3.5"/>
+        <limit effort="100.0" velocity="3.5"/>
         <axis xyz="-1 0 0"/>
         <parent link="base_link"/>
@@ -137,5 +136,5 @@
     <joint name="wheel_left_joint" type="continuous">
         <origin rpy="0 0 1.57079" xyz="-0.225 0.2625 -0.48"/>
-        <limit effort="10.0" velocity="3.5"/>
+        <limit effort="100.0" velocity="3.5"/>
         <axis xyz="1 0 0"/>
         <parent link="base_link"/>

Commit message: change absolute paths to meshes to  file://$(find sew_agv_description)

File: src/sew_agv_description/urdf/sew_agv_macro.urdf.xacro (robot description, xacro)
@@ -65,5 +65,5 @@
             <origin rpy="0 0 0" xyz="0 0 0"/>
             <geometry>
-                <mesh filename="/home/logilab/ros2_ws/src/sew_agv_description/meshes/visual/sew_maxo_mts_body.stl" scale="0.001 0.001 0.001"/>
+                <mesh filename="file://$(find sew_agv_description)/meshes/visual/sew_maxo_mts_body.stl" scale="0.001 0.001 0.001"/>
             </geometry>
             <material name="${tf_prefix}grey"/>
@@ -72,5 +72,5 @@
             <origin rpy=" 0 0 0" xyz="0 0 0"/>
             <geometry>
-                <mesh filename="/home/logilab/ros2_ws/src/sew_agv_description/meshes/collision/sew_maxo_mts_body.stl" scale="0.001 0.001 0.001"/>
+                <mesh filename="file://$(find sew_agv_description)/meshes/collision/sew_maxo_mts_body.stl" scale="0.001 0.001 0.001"/>
             </geometry>
             <material name="${tf_prefix}red"/>
@@ -92,5 +92,5 @@
             <origin rpy="0 0 0" xyz="0 0 0"/>
             <geometry>
-                <mesh filename="/home/logilab/ros2_ws/src/sew_agv_description/meshes/visual/sew_maxo_mts_front_wheel.stl" scale="0.001 0.001 0.001"/>
+                <mesh filename="file://$(find sew_agv_description)/meshes/visual/sew_maxo_mts_front_wheel.stl" scale="0.001 0.001 0.001"/>
             </geometry>
             <material name="${tf_prefix}black"/>
@@ -99,5 +99,5 @@
             <origin rpy="0 0 0" xyz="0 0 0"/>
             <geometry>
-                <mesh filename="/home/logilab/ros2_ws/src/sew_agv_description/meshes/visual/sew_maxo_mts_front_wheel.stl" scale="0.001 0.001 0.001"/>
+                <mesh filename="file://$(find sew_agv_description)/meshes/visual/sew_maxo_mts_front_wheel.stl" scale="0.001 0.001 0.001"/>
             </geometry>
             <material name="${tf_prefix}red"/>
@@ -121,5 +121,5 @@
             <origin rpy="0 0 0" xyz="0 0 0"/>
             <geometry>
-                <mesh filename="/home/logilab/ros2_ws/src/sew_agv_description/meshes/visual/sew_maxo_mts_wheel.stl" scale="0.001 0.001 0.001"/>
+                <mesh filename="file://$(find sew_agv_description)/meshes/visual/sew_maxo_mts_wheel.stl" scale="0.001 0.001 0.001"/>
             </geometry>
             <material name="${tf_prefix}black"/>
@@ -128,5 +128,5 @@
             <origin rpy="0 0 0" xyz="0 0 0"/>
             <geometry>
-                <mesh filename="/home/logilab/ros2_ws/src/sew_agv_description/meshes/visual/sew_maxo_mts_wheel.stl" scale="0.001 0.001 0.001"/>
+                <mesh filename="file://$(find sew_agv_description)/meshes/visual/sew_maxo_mts_wheel.stl" scale="0.001 0.001 0.001"/>
             </geometry>
             <material name="${tf_prefix}red"/>
@@ -150,5 +150,5 @@
             <origin rpy="0 0 0" xyz="0 0 0"/>
             <geometry>
-                <mesh filename="/home/logilab/ros2_ws/src/sew_agv_description/meshes/visual/sew_maxo_mts_wheel.stl" scale="0.001 0.001 0.001"/>
+                <mesh filename="file://$(find sew_agv_description)/meshes/visual/sew_maxo_mts_wheel.stl" scale="0.001 0.001 0.001"/>
             </geometry>
             <material name="${tf_prefix}black"/>
@@ -157,5 +157,5 @@
             <origin rpy="0 0 0" xyz="0 0 0"/>
             <geometry>
-                <mesh filename="/home/logilab/ros2_ws/src/sew_agv_description/meshes/visual/sew_maxo_mts_wheel.stl" scale="0.001 0.001 0.001"/>
+                <mesh filename="file://$(find sew_agv_description)/meshes/visual/sew_maxo_mts_wheel.stl" scale="0.001 0.001 0.001"/>
             </geometry>
             <material name="${tf_prefix}red"/>
@@ -178,5 +178,5 @@
             <origin rpy="0 0 0" xyz="0 0 0"/>
             <geometry>
-                <mesh filename="/home/logilab/ros2_ws/src/sew_agv_description/meshes/visual/sew_maxo_mts_lidar.stl" scale="0.001 0.001 0.001"/>
+                <mesh filename="file://$(find sew_agv_description)/meshes/visual/sew_maxo_mts_lidar.stl" scale="0.001 0.001 0.001"/>
             </geometry>
             <material name="${tf_prefix}yellow"/>
@@ -185,5 +185,5 @@
             <origin rpy="0 0 0" xyz="0 0 0"/>
             <geometry>
-                <mesh filename="/home/logilab/ros2_ws/src/sew_agv_description/meshes/visual/sew_maxo_mts_lidar.stl" scale="0.001 0.001 0.001"/>
+                <mesh filename="file://$(find sew_agv_description)/meshes/visual/sew_maxo_mts_lidar.stl" scale="0.001 0.001 0.001"/>
             </geometry>
         </collision>

Commit message: redefine inertia properties

File: src/sew_agv_description/urdf/sew_agv_macro.urdf.xacro (robot description, xacro)
@@ -60,5 +60,5 @@
             <mass value="250"/> <!--in kg-->
             <origin rpy="0 0 0" xyz="0 0 0"/>
-            <inertia ixx="1.0" ixy="0.0" ixz="0.0" iyy="1.0" iyz="0.0" izz="1.0"/> <!--not realistic!-->
+            <inertia ixx="3.82" ixy="0.0" ixz="0.48" iyy="4.11" iyz="0.0" izz="3.29"/> <!--not realistic!-->
         </inertial>
         <visual>
@@ -87,5 +87,5 @@
         <inertial>
             <mass value="2"/>
-            <inertia ixx="1.0" ixy="0.0" ixz="0.0" iyy="1.0" iyz="0.0" izz="1.0"/> <!--not realistic!-->
+            <inertia ixx="0.0" ixy="0.0" ixz="0.0" iyy="1.0" iyz="0.0" izz="1.0"/> <!--not realistic!-->
         </inertial>
         <visual>
@@ -116,5 +116,5 @@
             <origin rpy="0 0 0" xyz="0 0 0"/>
             <mass value="2"/>
-            <inertia ixx="1.0" ixy="0.0" ixz="0.0" iyy="1.0" iyz="0.0" izz="1.0"/> <!--not realistic!-->
+            <inertia ixx="0.0" ixy="0.0" ixz="0.0" iyy="1.0" iyz="0.0" izz="1.0"/> <!--not realistic!-->
         </inertial>
         <visual>

Commit message: moved <material name="${tf_prefix}red"/> from outside the </collision> tag inside the tag

File: src/sew_agv_description/urdf/sew_agv_macro.urdf.xacro (robot description, xacro)
@@ -119,5 +119,5 @@
         </collision>
     </link>
-    <!--right back wheel / axis shold match the rotation axis of the wheel-->
+    <!--right back wheel / axis should match the rotation axis of the wheel-->
     <joint name="${tf_prefix}wheel_right_joint" type="continuous">
         <origin rpy="0 0 -1.57079" xyz="-0.225 -0.2625 -0.48"/>
@@ -148,5 +148,5 @@
         </collision>
     </link>
-    <!--left back wheel / axis shold match the rotation axis of the wheel-->
+    <!--left back wheel / axis should match the rotation axis of the wheel-->
     <joint name="${tf_prefix}wheel_left_joint" type="continuous">
         <origin rpy="0 0 1.57079" xyz="-0.225 0.2625 -0.48"/>
@@ -202,6 +202,6 @@
                 <mesh filename="file://$(find sew_agv_description)/meshes/visual/sew_maxo_mts_lidar.stl" scale="0.001 0.001 0.001"/>
             </geometry>
-        </collision>
-        <material name="${tf_prefix}red"/>
+            <material name="${tf_prefix}red"/>
+        </collision>
     </link>
   </xacro:macro>
